File: Section B - TItle B.kicad_sch (KiCad schematic)
At the start: 0 parts

Commit message: First draft of schematic
Parts:
- added C19, C21, C22: 0.1uF, Capacitor_SMD:C_0603_1608Metric, symbol Device:C
- added C20: 4.7uF, Capacitor_SMD:C_0603_1608Metric, symbol Device:C
- added J2: CE, Connector_PinHeader_2.54mm:PinHeader_1x02_P2.54mm_Vertical, symbol Connector:Conn_01x02_Pin
- added J3: Conn_01x03_Pin, Connector_PinSocket_2.54mm:PinSocket_1x03_P2.54mm_Vertical, symbol Connector:Conn_01x03_Pin
- added R10, R11, R12, R9: 4.7kR, Resistor_SMD:R_0402_1005Metric, symbol Device:R
- added U2: TLV73333PDBV, Package_TO_SOT_SMD:SOT-23-5, symbol Regulator_Linear:TLV73333PDBV
- added U3: MSPM0C1104SDSGR, Package_TO_SOT_SMD:TSOT-23-8, symbol solar_station:MSPM0C1104SDSGR
Connections:
- new net: C19.2, J2.2 (Pin_2), U2.1 (IN), U2.3 (EN)
- new net: R11.1, U3.8 (PA24/A3)
- new net: J3.2 (Pin_2), U3.6 (PA19/SWDIO)
- new net: J3.3 (Pin_3), U3.7 (PA20/A6/SWCLK)
- new net +3V3: C20.2, C21.2, C22.2, R10.1, R12.2, R9.1, U2.5 (OUT), U3.4 (VDD)
- new net GND: C19.1, C20.1, C21.1, C22.1, R11.2, U2.2 (GND), U3.3 (VSS), U3.9 (EPAD)
- new net INT_N: R10.2, U3.1 (PA27/A0)
- new net REGN: J2.1 (Pin_1)
- new net SCL: J3.1 (Pin_1), R9.2, U3.2 (PA1/NRST)
- new net SDA: R12.1, U3.5 (PA0)
Other:
- title: Sheet Title B -> MCU
