File: solar_smart_station.kicad_pcb (KiCad board)
At the start: 6 copper layers, 0 parts

Commit message: First draft of schematic
Parts:
- added C1: 2.2uF, Capacitor_SMD:C_0805_2012Metric, F.Cu at (52.2, 156.2)
- added C10: 0.1uF, Capacitor_SMD:C_0603_1608Metric, F.Cu at (50.9, 168.3)
- added C11: 10uF, Capacitor_SMD:C_1206_3216Metric, F.Cu at (32.8, 157.3)
- added C12: 10uF, Capacitor_SMD:C_1206_3216Metric, F.Cu at (32.8, 160.7)
- added C13: 10uF, Capacitor_SMD:C_1206_3216Metric, F.Cu at (32.8, 164.1)
- added C14: 10uF, Capacitor_SMD:C_1206_3216Metric, F.Cu at (32.8, 167.4)
- added C15: 10uF, Capacitor_SMD:C_1206_3216Metric, F.Cu at (32.8, 170.8)
- added C16: 10uF, Capacitor_SMD:C_1206_3216Metric, F.Cu at (32.8, 174.1)
- added C17: 10uF, Capacitor_SMD:C_1206_3216Metric, F.Cu at (32.8, 177.4)
- added C18: 10uF, Capacitor_SMD:C_1206_3216Metric, F.Cu at (32.8, 180.8)
- added C19: 0.1uF, Capacitor_SMD:C_0603_1608Metric, F.Cu at (67.2, 173.5)
- added C2: 0.1uF, Capacitor_SMD:C_0603_1608Metric, F.Cu at (50.9, 160.8)
- added C20: 4.7uF, Capacitor_SMD:C_0603_1608Metric, F.Cu at (69.0, 150.2)
- added C21: 0.1uF, Capacitor_SMD:C_0603_1608Metric, F.Cu at (69.0, 152.7)
- added C22: 0.1uF, Capacitor_SMD:C_0603_1608Metric, F.Cu at (67.2, 171.0)
- added C3: 10uF, Capacitor_SMD:C_1206_3216Metric, F.Cu at (32.8, 150.7)
- added C4: 10uF, Capacitor_SMD:C_1206_3216Metric, F.Cu at (32.8, 154.0)
- added C5: 47nF, Capacitor_SMD:C_0402_1005Metric, F.Cu at (54.5, 171.1)
- added C6: 4.7uF, Capacitor_SMD:C_0603_1608Metric, F.Cu at (50.9, 163.3)
- added C7: 47nF, Capacitor_SMD:C_0402_1005Metric, F.Cu at (54.5, 173.0)
- added C8: 1nF, Capacitor_SMD:C_0402_1005Metric, F.Cu at (54.5, 175.0)
- added C9: 0.1uF, Capacitor_SMD:C_0603_1608Metric, F.Cu at (50.9, 165.8)
- added J1: CE, Connector_PinHeader_2.54mm:PinHeader_1x02_P2.54mm_Vertical, F.Cu at (55.2, 161.8)
- added J2: CE, Connector_PinHeader_2.54mm:PinHeader_1x02_P2.54mm_Vertical, F.Cu at (62.9, 167.4)
- added J3: Conn_01x03_Pin, Connector_PinSocket_2.54mm:PinSocket_1x03_P2.54mm_Vertical, F.Cu at (61.8, 151.3)
- added J4: JST_VH_B2P_3.96mm, Connector_JST:JST_VH_B2P-VH_1x02_P3.96mm_Vertical, F.Cu at (78.8, 156.4)
- added J5: JST_VH_B2P_3.96mm, Connector_JST:JST_VH_B2P-VH_1x02_P3.96mm_Vertical, F.Cu at (89.1, 156.4)
- added J6: JST_VH_B3P_3.96mm, Connector_JST:JST_VH_B3P-VH_1x03_P3.96mm_Vertical, F.Cu at (78.8, 166.9)
- added L1: 1uH, Inductor_SMD:L_Bourns_SRP7028A_7.3x6.6mm, F.Cu at (43.5, 174.2)
- added R1: 2R-1W, Resistor_SMD:R_2010_5025Metric, F.Cu at (42.2, 180.3)
- added R10: 4.7kR, Resistor_SMD:R_0402_1005Metric, F.Cu at (65.5, 152.0)
- added R11: 4.7kR, Resistor_SMD:R_0402_1005Metric, F.Cu at (65.5, 153.9)
- added R12: 4.7kR, Resistor_SMD:R_0402_1005Metric, F.Cu at (65.5, 155.9)
- added R2: 4.7kR, Resistor_SMD:R_0402_1005Metric, F.Cu at (37.1, 160.5)
- added R3: 5.24kR, Resistor_SMD:R_0402_1005Metric, F.Cu at (37.1, 162.5)
- added R4: 30.31kR, Resistor_SMD:R_0402_1005Metric, F.Cu at (37.1, 164.5)
- added R5: 6.04kR, Resistor_SMD:R_0402_1005Metric, F.Cu at (37.1, 166.5)
- added R6: 100R, Resistor_SMD:R_0402_1005Metric, F.Cu at (37.1, 168.5)
- added R7: 127kR, Resistor_SMD:R_0402_1005Metric, F.Cu at (37.1, 170.5)
- added R8: 100kR, Resistor_SMD:R_0402_1005Metric, F.Cu at (37.1, 172.5)
- added R9: 4.7kR, Resistor_SMD:R_0402_1005Metric, F.Cu at (65.5, 150.0)
- added TP1: QON, Connector_PinHeader_2.54mm:PinHeader_1x01_P2.54mm_Vertical, F.Cu at (50.8, 172.4)
- added TP2: Thermistor, Connector_PinHeader_2.54mm:PinHeader_1x01_P2.54mm_Vertical, F.Cu at (50.8, 177.0)
- added U1: BQ25672RQMR, solar_station:RQM0029A-MFG, F.Cu at (53.4, 151.8)
- added U2: TLV73333PDBV, Package_TO_SOT_SMD:SOT-23-5, F.Cu at (67.8, 167.5)
- added U3: MSPM0C1104SDSGR, Package_TO_SOT_SMD:TSOT-23-8, F.Cu at (66.7, 159.3)
