File: solar_smart_station.kicad_pcb (KiCad board)
At the start: 4 copper layers, 57.8 x 39.5 mm, 92 parts, among them J1 Conn_01x02_Pin, J2 LDO_EN, J3 Conn_01x05_Pin, J4 Thermistor_1, J5 Thermistor_2, Q1 AO3400A, Q2 AO3400A, U1 BQ25672RQMR, U2 TLV73333PDBV, U3 MSPM0C1104SDSGR, U4 BQ7791500PWR, U5 CSD25402Q3A

Commit message: Update Outputs (release)
Other:
- board text added: "0.02mm"
- board text added: "0.035mm (1.00oz)"
- board text added: "0.07mm (2.00oz)"
- board text added: "0.1mm"
- board text added: "1.21mm"
- board text added: "B.Mask"
- board text added: "B.Paste"
- board text added: "B.Silkscreen"
- board text added: "Copper"
- board text added: "Core"
- board text added: "Dielectric"
- board text added: "Direct Printing"
- board text added: "F.Mask"
- board text added: "F.Paste"
- board text added: "F.Silkscreen"
- board text added: "FR4"
- board text added: "FR4_7628"
- board text added: "GBR"
- board text added: "Gerber"
- board text added: "L1 (Sig, PWR)"
- board text added: "L2 (GND)"
- board text added: "L3 (GND)"
- board text added: "L4 (Sig, PWR)"
- board text added: "Layer"
- board text added: "Legend"
- board text added: "Material"
- board text added: "Note: external layer thicknesses are specified after plating"
- board text added: "Paste Mask"
- board text added: "Plane"
- board text added: "Prepreg"
- board text added: "Signal"
- board text added: "Solder Mask"
- board text added: "Solder Resist"
- board text added: "Thickness"
- board text added: "Total thickness: 1.66mm"
- board text added: "Type"
